File: pdu.kicad_sch (KiCad schematic)
At the start: 4 parts

Commit message: Third revision
Signed-off-by: Roman Ondráček <ondracek.roman@centrum.cz>
Other:
- removed sheet Ethernet
- sheet ESP32 ports: added CRITICAL; removed EMAC_RST, RMII_CLK, RMII_CRS_DV, RMII_RXD0, RMII_RXD1, RMII_TXD0, RMII_TXD1, RMII_TXEN, SMI_MDC, SMI_MDIO
- sheet Outputs ports: added CRITICAL; removed none
Changed lines of the file:
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@@
   (title_block
     (title "PDU with Consumption Metering Function for SBCs")
-    (date "2023-04-17")
-    (rev "2")
+    (date "2023-05-03")
+    (rev "1.0 rev 3")
   )
   (junction (at 120.65 143.51) (diameter 0) (color 0 0 0 0)
@@
     (stroke (width 0) (type default))
   )
-  (wire (pts (xy 144.78 97.79) (xy 156.21 97.79))
-    (stroke (width 0) (type default))
-  )
-  (wire (pts (xy 144.78 115.57) (xy 156.21 115.57))
-    (stroke (width 0) (type default))
-  )
   (wire (pts (xy 187.96 95.25) (xy 196.85 95.25))
     (stroke (width 0) (type default))
   )
-  (wire (pts (xy 144.78 85.09) (xy 156.21 85.09))
-    (stroke (width 0) (type default))
-  )
   (wire (pts (xy 187.96 115.57) (xy 196.85 115.57))
     (stroke (width 0) (type default))
@@
     (stroke (width 0) (type default))
   )
-  (wire (pts (xy 144.78 102.87) (xy 156.21 102.87))
-    (stroke (width 0) (type default))
-  )
   (wire (pts (xy 187.96 101.6) (xy 196.85 101.6))
     (stroke (width 0) (type default))
@@
     (stroke (width 0) (type default))
   )
-  (wire (pts (xy 144.78 92.71) (xy 156.21 92.71))
-    (stroke (width 0) (type default))
-  )
   (wire (pts (xy 120.65 151.13) (xy 120.65 158.75))
     (stroke (width 0) (type default))
@@
     (stroke (width 0) (type default))
   )
-  (wire (pts (xy 144.78 95.25) (xy 156.21 95.25))
-    (stroke (width 0) (type default))
-  )
   (wire (pts (xy 120.65 151.13) (xy 123.19 151.13))
     (stroke (width 0) (type default))
@@
     (stroke (width 0) (type default))
   )
-  (wire (pts (xy 144.78 90.17) (xy 156.21 90.17))
-    (stroke (width 0) (type default))
-  )
   (wire (pts (xy 187.96 106.68) (xy 196.85 106.68))
     (stroke (width 0) (type default))
@@
     (stroke (width 0) (type default))
   )
-  (wire (pts (xy 144.78 107.95) (xy 156.21 107.95))
-    (stroke (width 0) (type default))
-  )
   (wire (pts (xy 120.65 158.75) (xy 120.65 161.29))
     (stroke (width 0) (type default))
   )
-  (wire (pts (xy 144.78 113.03) (xy 156.21 113.03))
-    (stroke (width 0) (type default))
-  )
   (wire (pts (xy 120.65 135.89) (xy 123.19 135.89))
     (stroke (width 0) (type default))
   )
-  (wire (pts (xy 144.78 105.41) (xy 156.21 105.41))
+  (wire (pts (xy 187.96 119.38) (xy 196.85 119.38))
     (stroke (width 0) (type default))
   )
@@
   (symbol (lib_id "power:GND") (at 120.65 161.29 0) (unit 1)
     (in_bom yes) (on_board yes) (dnp no) (fields_autoplaced)
-    (property "Reference" "#PWR097" (at 120.65 167.64 0)
+    (property "Reference" "#PWR01" (at 120.65 167.64 0)
       (effects (font (size 1.27 1.27)) hide)
     )
@@
     (pin "1")
     (instances
-      (project "pdu_new"
-        (path "/fae03d15-1958-4da4-90aa-55c91e006394"
-          (reference "#PWR097") (unit 1)
+      (project "pdu"
+        (path "/fae03d15-1958-4da4-90aa-55c91e006394"
+          (reference "#PWR01") (unit 1)
         )
       )
@@
     (pin "1")
     (instances
-      (project "pdu_new"
+      (project "pdu"
         (path "/fae03d15-1958-4da4-90aa-55c91e006394"
           (reference "H2") (unit 1)
@@
     (pin "1")
     (instances
-      (project "pdu_new"
+      (project "pdu"
         (path "/fae03d15-1958-4da4-90aa-55c91e006394"
           (reference "H1") (unit 1)
@@
     (pin "1")
     (instances
-      (project "pdu_new"
+      (project "pdu"
         (path "/fae03d15-1958-4da4-90aa-55c91e006394"
           (reference "H3") (unit 1)
@@
     (pin "1")
     (instances
-      (project "pdu_new"
+      (project "pdu"
         (path "/fae03d15-1958-4da4-90aa-55c91e006394"
           (reference "H4") (unit 1)
@@
     )
     (instances
-      (project "pdu_new"
+      (project "pdu"
         (path "/fae03d15-1958-4da4-90aa-55c91e006394" (page "2"))
       )
     )
   )
-  (sheet (at 196.85 82.55) (size 24.13 35.56) (fields_autoplaced)
+  (sheet (at 196.85 82.55) (size 24.13 39.37) (fields_autoplaced)
     (stroke (width 0.1524) (type solid))
     (fill (color 0 0 0 0.0000))
@@
       (effects (font (size 1.27 1.27)) (justify left bottom))
     )
-    (property "Sheetfile" "outputs.kicad_sch" (at 196.85 118.6946 0)
+    (property "Sheetfile" "outputs.kicad_sch" (at 196.85 122.5046 0)
       (effects (font (size 1.27 1.27)) (justify left top))
     )
@@
       (effects (font (size 1.27 1.27)) (justify left))
     )
-    (instances
-      (project "pdu_new"
+    (pin "CRITICAL" output (at 196.85 119.38 180)
+      (effects (font (size 1.27 1.27)) (justify left))
+    )
+    (instances
+      (project "pdu"
         (path "/fae03d15-1958-4da4-90aa-55c91e006394" (page "4"))
       )
     )
   )
-  (sheet (at 120.65 82.55) (size 24.13 35.56) (fields_autoplaced)
-    (stroke (width 0.1524) (type solid))
-    (fill (color 0 0 0 0.0000))
-    (property "Sheetname" "Ethernet" (at 120.65 81.8384 0)
-      (effects (font (size 1.27 1.27)) (justify left bottom))
-    )
-    (property "Sheetfile" "ethernet.kicad_sch" (at 120.65 118.6946 0)
-      (effects (font (size 1.27 1.27)) (justify left top))
-    )
-    (pin "SMI_MDC" input (at 144.78 113.03 0)
-      (effects (font (size 1.27 1.27)) (justify right))
-    )
-    (pin "RST" input (at 144.78 85.09 0)
-      (effects (font (size 1.27 1.27)) (justify right))
-    )
-    (pin "SMI_MDIO" bidirectional (at 144.78 115.57 0)
-      (effects (font (size 1.27 1.27)) (justify right))
-    )
-    (pin "RMII_RXD0" output (at 144.78 90.17 0)
-      (effects (font (size 1.27 1.27)) (justify right))
-    )
-    (pin "RMII_CLK" input (at 144.78 107.95 0)
-      (effects (font (size 1.27 1.27)) (justify right))
-    )
-    (pin "RMII_RXD1" output (at 144.78 92.71 0)
-      (effects (font (size 1.27 1.27)) (justify right))
-    )
-    (pin "RMII_CRS_DV" output (at 144.78 105.41 0)
-      (effects (font (size 1.27 1.27)) (justify right))
-    )
-    (pin "RMII_TXEN" input (at 144.78 102.87 0)
-      (effects (font (size 1.27 1.27)) (justify right))
-    )
-    (pin "RMII_TXD1" input (at 144.78 97.79 0)
-      (effects (font (size 1.27 1.27)) (justify right))
-    )
-    (pin "RMII_TXD0" input (at 144.78 95.25 0)
-      (effects (font (size 1.27 1.27)) (justify right))
-    )
-    (instances
-      (project "pdu_new"
-        (path "/fae03d15-1958-4da4-90aa-55c91e006394" (page "5"))
-      )
-    )
-  )
-  (sheet (at 156.21 82.55) (size 31.75 35.56) (fields_autoplaced)
+  (sheet (at 156.21 82.55) (size 31.75 39.37) (fields_autoplaced)
     (stroke (width 0.1524) (type solid))
     (fill (color 0 0 0 0.0000))
@@
       (effects (font (size 1.27 1.27)) (justify left bottom))
     )
-    (property "Sheetfile" "esp32.kicad_sch" (at 156.21 118.6946 0)
+    (property "Sheetfile" "esp32.kicad_sch" (at 156.21 122.5046 0)
       (effects (font (size 1.27 1.27)) (justify left top))
     )
@@
       (effects (font (size 1.27 1.27)) (justify right))
     )
-    (pin "SMI_MDIO" bidirectional (at 156.21 115.57 180)
-      (effects (font (size 1.27 1.27)) (justify left))
-    )
-    (pin "SMI_MDC" output (at 156.21 113.03 180)
-      (effects (font (size 1.27 1.27)) (justify left))
-    )
-    (pin "EMAC_RST" output (at 156.21 85.09 180)
-      (effects (font (size 1.27 1.27)) (justify left))
-    )
-    (pin "RMII_CLK" output (at 156.21 107.95 180)
-      (effects (font (size 1.27 1.27)) (justify left))
-    )
-    (pin "RMII_TXD0" output (at 156.21 95.25 180)
-      (effects (font (size 1.27 1.27)) (justify left))
-    )
-    (pin "RMII_TXD1" output (at 156.21 97.79 180)
-      (effects (font (size 1.27 1.27)) (justify left))
-    )
-    (pin "RMII_TXEN" output (at 156.21 102.87 180)
-      (effects (font (size 1.27 1.27)) (justify left))
-    )
-    (pin "RMII_CRS_DV" input (at 156.21 105.41 180)
-      (effects (font (size 1.27 1.27)) (justify left))
-    )
-    (pin "RMII_RXD0" input (at 156.21 90.17 180)
-      (effects (font (size 1.27 1.27)) (justify left))
-    )
-    (pin "RMII_RXD1" input (at 156.21 92.71 180)
-      (effects (font (size 1.27 1.27)) (justify left))
-    )
-    (instances
-      (project "pdu_new"
+    (pin "CRITICAL" input (at 187.96 119.38 0)
+      (effects (font (size 1.27 1.27)) (justify right))
+    )
+    (instances
+      (project "pdu"
         (path "/fae03d15-1958-4da4-90aa-55c91e006394" (page "3"))
       )
