File: outputs.kicad_sch (KiCad schematic)
At the start: 24 parts, among them J6 USB_A, J7 USB_A, U7 TPS2000C, U8 TPS2000C, U9 INA3221

Commit message: Second revision
Signed-off-by: Roman Ondráček <ondracek.roman@centrum.cz>
Parts:
- removed C24, C28: C, Capacitor_SMD:C_0402_1005Metric_Pad0.74x0.62mm_HandSolder, symbol Device:C
- removed C29, C30: 100n, Capacitor_SMD:C_0402_1005Metric_Pad0.74x0.62mm_HandSolder, symbol Device:C
- removed C31: 150u, Capacitor_Tantalum_SMD:CP_EIA-7343-31_Kemet-D_Pad2.25x2.55mm_HandSolder, symbol Device:C_Polarized
- removed R20, R21: 10k, Resistor_SMD:R_0402_1005Metric_Pad0.72x0.64mm_HandSolder, symbol Device:R
- removed R22: 10R, Resistor_SMD:R_0402_1005Metric_Pad0.72x0.64mm_HandSolder, symbol Device:R
- removed R23: R_Shunt, Resistor_SMD:R_Shunt_Ohmite_LVK12, symbol Device:R_Shunt
- added C24 (x3), C31, C32, C34, C37, C38, C40: 100n, Capacitor_SMD:C_0402_1005Metric_Pad0.74x0.62mm_HandSolder, symbol Device:C
- added C26: C, Capacitor_SMD:C_0402_1005Metric_Pad0.74x0.62mm_HandSolder, symbol Device:C
- added C35, C41: 150u, Capacitor_Tantalum_SMD:CP_EIA-7343-31_Kemet-D_Pad2.25x2.55mm_HandSolder, symbol Device:C_Polarized
- added D2 (x3): Green_LED, LED_SMD:LED_0603_1608Metric_Pad1.05x0.95mm_HandSolder, symbol Device:LED
- added D4 (x3): Amber_LED, LED_SMD:LED_0603_1608Metric_Pad1.05x0.95mm_HandSolder, symbol Device:LED
- added J6: USB_A, Connector_USB_custom.pretty:USB_A_GCT_USB1125-GF-B, symbol Connector:USB_A
- added R27, R32, R34, R36, R37, R42, R44, R46, R47, R7 (x3): 10k, Resistor_SMD:R_0402_1005Metric_Pad0.72x0.64mm_HandSolder, symbol Device:R
- added R29, R30, R40, R41: 10R, Resistor_SMD:R_0402_1005Metric_Pad0.72x0.64mm_HandSolder, symbol Device:R
- added R33, R43: 50m, Resistor_SMD:R_Shunt_Ohmite_LVK12, symbol Device:R_Shunt
- added R5 (x3): 100R, Resistor_SMD:R_0603_1608Metric_Pad0.98x0.95mm_HandSolder, symbol Device:R
- added R5 (x3): 100R, Resistor_SMD:R_0402_1005Metric_Pad0.72x0.64mm_HandSolder, symbol Device:R
- added SW1 (x3): SW_Push, Button_Switch_SMD:SW_Push_1P1T_NO_6x6mm_H9.5mm, symbol Switch:SW_Push
- added U7: TPS2000C, Package_SO:VSSOP-8_3.0x3.0mm_P0.65mm, symbol Power_Management:TPS2000C
- C27: renamed from C25; Mouser (none) -> https://cz.mouser.com/ProductDetail/187-CL21B104KCFSFNE
- C29: renamed from C26; Mouser (none) -> https://cz.mouser.com/ProductDetail/187-CL21B104KCFSFNE
- C30: renamed from C27; Mouser (none) -> https://cz.mouser.com/ProductDetail/581-TPSD157K010S0100
- J5: renamed from J6; footprint Connector_USB:USB_A_GCT_USB1125-GF-B -> Connector_USB_custom.pretty:USB_A_GCT_USB1125-GF-B; Mouser (none) -> https://cz.mouser.com/ProductDetail/640-USB1125-GF-B
- J7: footprint Connector_USB:USB_A_GCT_USB1125-GF-B -> Connector_USB_custom.pretty:USB_A_GCT_USB1125-GF-B; Mouser (none) -> https://cz.mouser.com/ProductDetail/640-USB1125-GF-B
- R19: renamed from R17; Mouser (none) -> https://cz.mouser.com/ProductDetail/667-ERJ-2RKF10R0X
- R20: renamed from R19; Mouser (none) -> https://cz.mouser.com/ProductDetail/667-ERJ-2RKF10R0X
- R22: renamed from R15; Mouser (none) -> https://cz.mouser.com/ProductDetail/652-CR0402FX-1002GLF
- R23: renamed from R18; value R_Shunt -> 50m
- R24: value 10R -> 10k; Mouser (none) -> https://cz.mouser.com/ProductDetail/652-CR0402FX-1002GLF
- R26: renamed from R16; Mouser (none) -> https://cz.mouser.com/ProductDetail/652-CR0402FX-1002GLF
- U6: renamed from U7; Mouser (none) -> https://cz.mouser.com/ProductDetail/595-TPS2000CDGNR
- U8: Mouser (none) -> https://cz.mouser.com/ProductDetail/595-TPS2000CDGNR
- U9: Mouser (none) -> https://cz.mouser.com/ProductDetail/595-INA3221AIRGVR
- renumbered C32 to C36
Connections:
- net +3V3: now also R32.1, R36.2, R42.1, R46.2, R7.1, R7.1, R7.1
- net +5V: now also C32.2, C38.2, U7.2 (IN), U7.3 (IN)
- net GND: now also C24.2, C24.2, C24.2, C32.1, C34.2, C35.2, C38.1, C40.2, C41.2, D2.1 (K), D2.1 (K), D2.1 (K), D4.1 (K), D4.1 (K), D4.1 (K), J6.4 (GND), J6.5 (Shield), R27.2, R37.2, R47.2, SW1.2, SW1.2, SW1.2, U7.1 (GND)
- net ~{SBC1_FLT}: now also R5.1
- net ~{SBC2_EN}: now also R36.1, U7.4 (~{EN}); no longer U8.4 (~{EN})
- net ~{SBC2_FLT}: now also R32.2, R5.1, U7.5 (~{FLT}); no longer U8.5 (~{FLT})
- net at J5.1 (VBUS): now also R23.4; no longer R23.1
- net at J5.2 (D-), J5.3 (D+): now also R24.2, R27.1
- net SBC1_POWER: now reaches R24.1
- net SBC1_POWER: now also C29.1, C30.1, R23.1, U6.6 (OUT), U6.7 (OUT), U6.8 (OUT), R5.1
- net at R20.1, R23.3: now also C26.2
- net IN2+: now reaches U9.15 (IN+2)
- net IN2+: now also R30.2
- net at R23.2: now also R19.1, C26.1; no longer R19.2
- net at J7.1 (VBUS): now also R43.4
- net at J7.2 (D-), J7.3 (D+): now also R44.2, R47.1
- net IN+1 renamed IN1+
- net IN+2 renamed IN3+
- net IN3+: now also R41.2; no longer R24.2
- net IN-1 renamed IN1-
- net IN1-: now also R19.2; no longer R19.1
- net IN-2 renamed IN2-
- net IN2-: now also R29.2; no longer U9.1 (IN-3)
- removed net USB1_PWR: C29.1, C30.1, R23.4, U6.6 (OUT), U6.7 (OUT), U6.8 (OUT)
- net USB2_PWR renamed SBC3_POWER
- net SBC3_POWER: now also C40.1, C41.1, R43.1, R44.1, R5.1
- new net: C31.2, R30.1, R33.3
- new net: J6.1 (VBUS), R33.4
- new net: J6.2 (D-), J6.3 (D+), R34.2, R37.1
- new net: D4.2 (A), R5.2 (x3)
- new net: C37.1, R40.1, R43.2
- new net: C37.2, R41.1, R43.3
- new net: D2.2 (A), R5.2 (x3)
- new net: C31.1, R29.1, R33.2
- new net IN3-: R40.2, U9.1 (IN-3)
- new net SBC1_BTN: C24.1, R7.2, SW1.1
- new net SBC2_BTN: C24.1, R7.2, SW1.1
- new net SBC2_POWER: C34.1, C35.1, R33.1, R34.1, R5.1, U7.6 (OUT), U7.7 (OUT), U7.8 (OUT)
- new net SBC3_BTN: C24.1, R7.2, SW1.1
- new net ~{SBC3_EN}: R46.1, U8.4 (~{EN})
- new net ~{SBC3_FLT}: R42.2, R5.1, U8.5 (~{FLT})
- no-connect marks 5 -> 4
Other:
- note added: "Current shunt and bus voltage sensor"
- note added: "Output 1"
- note added: "Output 2"
- note added: "Output 3"
- note added: "USB power switch"
- title: (none) -> PDU with Consumption Metering Function for SBCs
- moved on the sheet: C27, C29, C30, C36, J5, R19, R20, R22, R23, R26, U6, U9

Commit message: Third revision
Signed-off-by: Roman Ondráček <ondracek.roman@centrum.cz>
Parts:
- removed R20, R29, R30, R40, R41: 10R, Resistor_SMD:R_0402_1005Metric_Pad0.72x0.64mm_HandSolder, symbol Device:R
- removed R22, R24, R26, R27, R34, R42, R44, R46, R47, R7 (x3): 10k, Resistor_SMD:R_0402_1005Metric_Pad0.72x0.64mm_HandSolder, symbol Device:R
- added R18, R31: 10R, Resistor_SMD:R_0402_1005Metric_Pad0.72x0.64mm_HandSolder, symbol Device:R
- added R2: 10k, Resistor_SMD:R_0402_1005Metric_Pad0.72x0.64mm_HandSolder, symbol Device:R
- added RN1, RN2, RN3: 10k, Resistor_SMD:R_Array_Convex_4x0603, symbol Device:R_Pack04
- R32, R36, R37: value 10k -> 10R; Mouser https://cz.mouser.com/ProductDetail/652-CR0402FX-1002GLF -> https://cz.mouser.com/ProductDetail/667-ERJ-2RKF10R0X
- renumbered R23 to R20, R33 to R26, R43 to R33
Connections:
- net +3V3: now also R5.2, R5.2, R5.2, R2.1, RN1.5 (R4.2), RN1.6 (R3.2), RN1.7 (R2.2), RN1.8 (R1.2), RN2.5 (R4.2), RN2.6 (R3.2), RN2.7 (R2.2), RN2.8 (R1.2), RN3.5 (R4.2), RN3.6 (R3.2), RN3.7 (R2.2), RN3.8 (R1.2); no longer R32.1, R36.2
- net GND: no longer D4.1 (K), D4.1 (K), D4.1 (K), R37.2
- net IN1+: now also C26.2, R19.1, U9.2 (IN+3); no longer U9.12 (IN+1)
- net IN1-: now also C26.1, U9.1 (IN-3), R18.1; no longer R19.2, U9.11 (IN-1)
- net IN2+: now also C31.2, R37.1
- net IN2-: now also C31.1, R36.1
- net IN3+: now also C37.2, R32.1, U9.12 (IN+1); no longer U9.2 (IN+3)
- net IN3-: now also C37.1, U9.11 (IN-1), R31.1; no longer U9.1 (IN-3)
- net SBC1_BTN: now also RN1.1 (R1.1)
- net SBC2_BTN: now also RN2.3 (R3.1)
- net SBC3_BTN: now also RN3.3 (R3.1)
- net ~{SBC1_EN}: now also RN1.3 (R3.1)
- net ~{SBC1_FLT}: now also D4.1 (K), RN1.2 (R2.1); no longer R5.1
- net ~{SBC2_EN}: now also RN2.1 (R1.1); no longer R36.1
- net ~{SBC2_FLT}: now also D4.1 (K), RN2.2 (R2.1); no longer R32.2, R5.1
- net ~{SBC3_EN}: now also RN3.1 (R1.1)
- net ~{SBC3_FLT}: now also D4.1 (K), RN3.2 (R2.1); no longer R5.1
- net at R26.3: now also R37.2; no longer C31.2
- net at J6.2 (D-), J6.3 (D+): no longer R37.1
- net at R20.3: now also R19.2; no longer C26.2
- net at D4.2 (A): now also R5.1; no longer R5.2 (x3)
- net at R33.2: now also R31.2; no longer C37.1
- net at R33.3: now also R32.2; no longer C37.2
- net CRITICAL: now reaches U9.9 (CRITICAL)
- net CRITICAL: now also R2.2
- net at R26.2: now also R36.2; no longer C31.1
- new net: R18.2, R20.2
- no-connect marks 4 -> 6
Other:
- moved on the sheet: C24, C26, C31, C35, C37, D4, J6, J7, R26, R33, R5, SW1

Commit message: Fix third revision
Signed-off-by: Roman Ondráček <ondracek.roman@centrum.cz>
Parts:
- C24, C26, C27, C29, C31, C32, C34, C36, C37, C38, C40: Mouser https://cz.mouser.com/ProductDetail/187-CL21B104KCFSFNE -> https://cz.mouser.com/ProductDetail/81-GRM155R62A104KE4J
- R5: value 100R -> 430R
- R5: value 100R -> 1k; Mouser https://cz.mouser.com/ProductDetail/667-ERJ-UP3J431V -> https://cz.mouser.com/ProductDetail/603-RC0402FR-071KL
- RN1, RN2, RN3: Mouser (none) -> https://cz.mouser.com/ProductDetail/588-LVK12R050DER
- SW1: Mouser (none) -> https://cz.mouser.com/ProductDetail/653-B3FS-1000
Other:
- moved on the sheet: C36, R2, U9
