File: pdu.kicad_pcb (KiCad board)
At the start: 2 copper layers, 100 x 100 mm, 164 parts, among them J1 DC_Jack, J2 USB_B_Micro, J3 JTAG, J4 UART, J5 USB_A, J6 USB_A, J7 USB_A, J8 RJ45_Amphenol_RJMG1BD3B8K1ANR, Q1 FDD4243, Q2 BC846, Q3 BC846, SW1 SW_Push, SW2 SW_Push, SW3 SW_Push, SW4 SW_Push, SW5 SW_Push, U1 MAX17634BATP+, U10 CM1293A-02SO, U11 CM1293A-02SO, U12 LAN8720A, U2 TLV1117LV33DCYR, U3 CP2102N-A02-GQFN24, U4 ESP32-WROOM-32D, U5 MCP7940N-I/SN, U6 TPS2000C, U7 TPS2000C, U8 TPS2000C, U9 INA3221, Y1 32.765k

Commit message: Third revision
Signed-off-by: Roman Ondráček <ondracek.roman@centrum.cz>
Parts:
- removed C42: 1u, Capacitor_SMD:C_0603_1608Metric_Pad1.08x0.95mm_HandSolder
- removed C43: 470p, Capacitor_SMD:C_0402_1005Metric_Pad0.74x0.62mm_HandSolder
- removed C44, C45, C46, C47: 100n, Capacitor_SMD:C_0402_1005Metric_Pad0.74x0.62mm_HandSolder
- removed C48, C49, C50, C51: 22p, Capacitor_SMD:C_0402_1005Metric_Pad0.74x0.62mm_HandSolder
- removed J8: RJ45_Amphenol_RJMG1BD3B8K1ANR, Connector_RJ:RJ45_Amphenol_RJMG1BD3B8K1ANR
- removed JP1: JTAG_EN, Connector_PinHeader_2.54mm:PinHeader_1x02_P2.54mm_Vertical
- removed R23, R43: 50m, Resistor_SMD:R_Shunt_Ohmite_LVK12
- removed R24, R39, R42, R44, R46, R47: 10k, Resistor_SMD:R_0402_1005Metric_Pad0.72x0.64mm_HandSolder
- removed R25, R45: 100R, Resistor_SMD:R_0603_1608Metric_Pad0.98x0.95mm_HandSolder
- removed R28, R38, R48: 100R, Resistor_SMD:R_0402_1005Metric_Pad0.72x0.64mm_HandSolder
- removed R40, R41: 10R, Resistor_SMD:R_0402_1005Metric_Pad0.72x0.64mm_HandSolder
- removed R49, R50, R51, R52: 49.9R, Resistor_SMD:R_0402_1005Metric_Pad0.72x0.64mm_HandSolder
- removed R53: 12.1k, Resistor_SMD:R_0402_1005Metric_Pad0.72x0.64mm_HandSolder
- removed R54, R55: 270R, Resistor_SMD:R_0402_1005Metric_Pad0.72x0.64mm_HandSolder
- removed U10, U11: CM1293A-02SO, Package_SO:SC-74-6_1.5x2.9mm_P0.95mm
- removed U12: LAN8720A, Package_DFN_QFN:QFN-24-1EP_4x4mm_P0.5mm_EP2.6x2.6mm
- added RN3: 10k, Resistor_SMD:R_Array_Convex_4x0603, B.Cu at (105.2, 77.7)
- BT1: value Battery_Cell -> CR2032; moved to F.Cu
- C15, C18, D9: moved to F.Cu
- C19, C21, C36, R9, U5, U9, Y1: moved to B.Cu
- C22: value 6.8p -> 100n; moved to B.Cu
- C23: value 100n -> 6.8p; moved to B.Cu
- L1: footprint Inductor_SMD:L_Coilcraft_XAL6060-XXX -> Inductor_SMD:L_Bourns_SRP1245A
- R10: value 3k3 -> 22.1k
- R11: value 22.1k -> 47.5k
- R12: value 47.5k -> 10k
- R13: value 10k -> 470; moved to F.Cu
- R14: value 1k -> 470
- R15: value 1k -> 10k
- R18, R31, R32, R36, R37: value 10k -> 10R; moved to F.Cu
- R20: value 10R -> 50m; footprint Resistor_SMD:R_0402_1005Metric_Pad0.72x0.64mm_HandSolder -> Resistor_SMD:R_Shunt_Ohmite_LVK12
- R21, R27, R34: value 10k -> 100R; footprint Resistor_SMD:R_0402_1005Metric_Pad0.72x0.64mm_HandSolder -> Resistor_SMD:R_0603_1608Metric_Pad0.98x0.95mm_HandSolder
- R22: value 10k -> 100R
- R26: value 10k -> 50m; footprint Resistor_SMD:R_0402_1005Metric_Pad0.72x0.64mm_HandSolder -> Resistor_SMD:R_Shunt_Ohmite_LVK12; moved to F.Cu
- R29: value 10R -> 100R; moved to B.Cu
- R30: value 10R -> 10k; moved to B.Cu
- R35: footprint Resistor_SMD:R_0603_1608Metric_Pad0.98x0.95mm_HandSolder -> Resistor_SMD:R_0402_1005Metric_Pad0.72x0.64mm_HandSolder; moved to B.Cu
- R4, R5: value 100R -> 430R
- R7: value 10k -> 1k; moved to F.Cu
- R8: value 1k -> 3k3
- RN1, RN2: value 100R -> 10k
- U3: value CP2102N-A02-GQFN24 -> ESP32-WROOM-32D; footprint Package_DFN_QFN:QFN-24-1EP_4x4mm_P0.5mm_EP2.6x2.6mm -> RF_Module:ESP32-WROOM-32D
- U4: value ESP32-WROOM-32D -> CP2102N-Axx-xQFN28; footprint RF_Module:ESP32-WROOM-32 -> Package_DFN_QFN:QFN-28-1EP_5x5mm_P0.5mm_EP3.35x3.35mm; moved to F.Cu
- moved R7 78.7 mm to (48.0, 33.2), turned to 180 degrees
- moved H1 77.4 mm to (40.0, 40.0)
- moved R18 73.2 mm to (44.8, 104.2), turned to 180 degrees
- moved U3 66.2 mm to (104.1, 64.3), turned to 90 degrees
- moved H3 65.4 mm to (50.0, 90.0)
- moved H4 65.3 mm to (90.0, 90.0)
- moved R22 64.4 mm to (48.2, 115.2), turned to -90 degrees
- moved U4 63.3 mm to (52.6, 34.1), turned to -90 degrees
- moved R30 61.2 mm to (98.8, 50.8), turned to -90 degrees
- moved R21 59.1 mm to (55.8, 116.1), turned to 90 degrees
- moved R35 51.0 mm to (108.2, 115.3), turned to -90 degrees
- moved R27 50.9 mm to (85.2, 115.8), turned to 90 degrees
- moved R8 49.6 mm to (97.2, 50.8), turned to -90 degrees
- moved SW2 49.5 mm to (114.5, 27.0)
- moved C25 49.5 mm to (114.5, 33.0)
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Connections:
- C19 pad 1: GND -> +3V3
- C19 pad 2: +3V3 -> GND
- C20 pad 1: +3V3 -> GND
- C20 pad 2: GND -> +3V3
- C22 pad 1: Net-(U5-X2) -> +3V3
- C23 pad 1: +3V3 -> Net-(U5-X2)
- C26 pad 1: Net-(C26-Pad1) -> /Outputs/IN1-
- C26 pad 2: Net-(C26-Pad2) -> /Outputs/IN1+
- C28 pad 1: /ESP32/MTCK -> /ESP32/SBC1_BTN
- C31 pad 1: Net-(C31-Pad1) -> /Outputs/IN2-
- C31 pad 2: Net-(C31-Pad2) -> /Outputs/IN2+
- C33 pad 1: /ESP32/MTDI -> /ESP32/SBC2_BTN
- C37 pad 1: Net-(C37-Pad1) -> /Outputs/IN3-
- C37 pad 2: Net-(C37-Pad2) -> /Outputs/IN3+
- C39 pad 1: /ESP32/MTMS -> /ESP32/SBC3_BTN
- D10 pad 1: GND -> /ESP32/~{SBC1_FLT}
- D12 pad 1: GND -> /ESP32/~{SBC2_FLT}
- D14 pad 1: GND -> /ESP32/~{SBC3_FLT}
- R10 pad 1: +3V3 -> Net-(U4-VBUS)
- R10 pad 2: /ESP32/SCL -> VBUS
- R11 pad 1: Net-(U3-VBUS) -> Net-(U4-VBUS)
- R11 pad 2: VBUS -> GND
- R12 pad 1: Net-(U3-VBUS) -> Net-(U4-~{SUSPEND})
- R13 pad 1: Net-(U3-~{SUSPEND}) -> +3V3
- R13 pad 2: GND -> Net-(D7-A)
- R14 pad 2: Net-(D7-A) -> Net-(D8-A)
- R15 pad 1: +3V3 -> Net-(D9-K)
- R15 pad 2: Net-(D8-A) -> Net-(U5-VBAT)
- R16 pad 1: Net-(D9-K) -> /ESP32/~{DTR}
- R16 pad 2: Net-(U5-VBAT) -> Net-(Q2-B)
- R17 pad 1: /ESP32/~{DTR} -> /ESP32/~{RTS}
- R17 pad 2: Net-(Q2-B) -> Net-(Q3-B)
- R18 pad 1: /ESP32/~{RTS} -> /Outputs/IN1-
- R18 pad 2: Net-(Q3-B) -> Net-(R18-Pad2)
- R19 pad 1: Net-(C26-Pad1) -> /Outputs/IN1+
- R19 pad 2: /Outputs/IN1- -> Net-(R19-Pad2)
- R20 pad 1: Net-(C26-Pad2) -> /Outputs/SBC1_POWER
- R20 pad 2: /Outputs/IN1+ -> Net-(R18-Pad2)
- R21 pad 1: +3V3 -> Net-(D10-A)
- R21 pad 2: /ESP32/MTCK -> +3V3
- R22 pad 1: +3V3 -> /Outputs/SBC1_POWER
- R22 pad 2: /ESP32/~{SBC1_FLT} -> Net-(D11-A)
- R26 pad 1: /ESP32/~{SBC1_EN} -> /Outputs/SBC2_POWER
- R26 pad 2: +3V3 -> Net-(R26-Pad2)
- R27 pad 1: Net-(J5-D+) -> Net-(D12-A)
- R27 pad 2: GND -> +3V3
- R29 pad 1: Net-(C31-Pad1) -> /Outputs/SBC2_POWER
- R29 pad 2: /Outputs/IN2- -> Net-(D13-A)
- R30 pad 1: Net-(C31-Pad2) -> +3V3
- R30 pad 2: /Outputs/IN2+ -> /ESP32/CRITICAL
- R31 pad 1: +3V3 -> /Outputs/IN3-
- R31 pad 2: /ESP32/MTDI -> Net-(R31-Pad2)
- R32 pad 1: +3V3 -> /Outputs/IN3+
- R32 pad 2: /ESP32/~{SBC2_FLT} -> Net-(R32-Pad2)
- R33 pad 1: /Outputs/SBC2_POWER -> /Outputs/SBC3_POWER
- R33 pad 2: Net-(C31-Pad1) -> Net-(R31-Pad2)
- R33 pad 3: Net-(C31-Pad2) -> Net-(R32-Pad2)
- R33 pad 4: Net-(J6-VBUS) -> Net-(J7-VBUS)
- R34 pad 1: /Outputs/SBC2_POWER -> Net-(D14-A)
- R34 pad 2: Net-(J6-D+) -> +3V3
- R35 pad 1: /ESP32/~{SBC2_FLT} -> /Outputs/SBC3_POWER
- R35 pad 2: Net-(D12-A) -> Net-(D15-A)
- R36 pad 1: /ESP32/~{SBC2_EN} -> /Outputs/IN2-
- R36 pad 2: +3V3 -> Net-(R26-Pad2)
- R37 pad 1: Net-(J6-D+) -> /Outputs/IN2+
- R37 pad 2: GND -> Net-(R26-Pad3)
- R7 pad 1: +3V3 -> Net-(U4-~{RST})
- R7 pad 2: /ESP32/~{JTAG_EN} -> +3V3
- R8 pad 1: Net-(U3-~{RST}) -> +3V3
- R8 pad 2: +3V3 -> /ESP32/SDA
- R9 pad 2: /ESP32/SDA -> /ESP32/SCL
- RN1 pad 1: /Ethernet/TXD1 -> /ESP32/SBC1_BTN
- RN1 pad 2: /Ethernet/TXD0 -> /ESP32/~{SBC1_FLT}
- RN1 pad 3: /Ethernet/TXEN -> /ESP32/~{SBC1_EN}
- RN1 pad 5: unconnected-(RN1-R4.2-Pad5) -> +3V3
- RN1 pad 6: /ESP32/RMII_TXEN -> +3V3
- RN1 pad 7: /ESP32/RMII_TXD0 -> +3V3
- RN1 pad 8: /ESP32/RMII_TXD1 -> +3V3
- RN2 pad 1: /ESP32/RMII_CLK -> /ESP32/~{SBC2_EN}
- RN2 pad 2: /ESP32/RMII_RXD1 -> /ESP32/~{SBC2_FLT}
- RN2 pad 3: /ESP32/RMII_RXD0 -> /ESP32/SBC2_BTN
- RN2 pad 4: /ESP32/RMII_CRS_DV -> unconnected-(RN2-R4.1-Pad4)
- RN2 pad 5: /Ethernet/CRS_DV -> +3V3
- RN2 pad 6: /Ethernet/RXD0 -> +3V3
- RN2 pad 7: /Ethernet/RXD1 -> +3V3
- RN2 pad 8: /Ethernet/REF_CLK -> +3V3
- SW3 pad 1: /ESP32/MTCK -> /ESP32/SBC1_BTN
- SW4 pad 1: /ESP32/MTDI -> /ESP32/SBC2_BTN
- SW5 pad 1: /ESP32/MTMS -> /ESP32/SBC3_BTN
- U3 pad 1: unconnected-(U3-~{RI}/CLK-Pad1) -> GND
- U3 pad 10: unconnected-(U3-NC-Pad10) -> /ESP32/~{SBC2_FLT}
- U3 pad 11: unconnected-(U3-~{WAKEUP}/GPIO.3-Pad11) -> /ESP32/~{SBC2_EN}
- U3 pad 13: Net-(D8-K) -> /ESP32/MTMS
- U3 pad 14: Net-(D7-K) -> /ESP32/MTDI
- U3 pad 15: Net-(U3-~{SUSPEND}) -> GND
- U3 pad 16: unconnected-(U3-NC-Pad16) -> /ESP32/MTCK
- U3 pad 19: /ESP32/~{RTS} -> unconnected-(U3-SCS/CMD-Pad19)
- U3 pad 2: GND -> +3V3
- U3 pad 20: /ESP32/DEBUG_RX -> unconnected-(U3-SCK/CLK-Pad20)
- U3 pad 21: /ESP32/DEBUG_TX -> unconnected-(U3-SDO/SD0-Pad21)
- U3 pad 23: /ESP32/~{DTR} -> /ESP32/MTDO
- U3 pad 25: GND -> /ESP32/BTN
- U3 pad 3: /ESP32/USB_D+ -> /ESP32/EN
- U3 pad 4: /ESP32/USB_D- -> unconnected-(U3-SENSOR_VP-Pad4)
- U3 pad 5: +3V3 -> unconnected-(U3-SENSOR_VN-Pad5)
- U3 pad 6: +3V3 -> /ESP32/SBC3_BTN
- U3 pad 7: +3V3 -> /ESP32/~{SBC3_FLT}
- U3 pad 8: Net-(U3-VBUS) -> /ESP32/~{SBC3_EN}
- U3 pad 9: Net-(U3-~{RST}) -> /ESP32/SBC2_BTN
- U4 pad 1: GND -> unconnected-(U4-~{DCD}-Pad1)
- U4 pad 10: /ESP32/RMII_RXD0 -> unconnected-(U4-NC-Pad10)
- U4 pad 11: /ESP32/RMII_RXD1 -> Net-(U4-~{SUSPEND})
- U4 pad 12: /ESP32/RMII_CRS_DV -> unconnected-(U4-SUSPEND-Pad12)
- U4 pad 13: /ESP32/MTMS -> unconnected-(U4-CHREN-Pad13)
- U4 pad 14: /ESP32/MTDI -> unconnected-(U4-CHR1-Pad14)
- U4 pad 15: GND -> unconnected-(U4-CHR0-Pad15)
- U4 pad 16: /ESP32/MTCK -> unconnected-(U4-~{WAKEUP}/GPIO.3-Pad16)
- U4 pad 18: unconnected-(U4-SWP/SD3-Pad18) -> Net-(D8-K)
- U4 pad 19: unconnected-(U4-SCS/CMD-Pad19) -> Net-(D7-K)
- U4 pad 2: +3V3 -> unconnected-(U4-~{RI}/CLK-Pad2)
- U4 pad 23: /ESP32/MTDO -> unconnected-(U4-~{CTS}-Pad23)
- U4 pad 24: unconnected-(U4-IO2-Pad24) -> /ESP32/~{RTS}
- U4 pad 25: /ESP32/BTN -> /ESP32/DEBUG_RX
- U4 pad 26: /ESP32/SDA -> /ESP32/DEBUG_TX
- U4 pad 27: /ESP32/RMII_CLK -> unconnected-(U4-~{DSR}-Pad27)
- U4 pad 28: /ESP32/EMAC_RST -> /ESP32/~{DTR}
- U4 pad 29: /ESP32/SCL -> GND
- U4 pad 3: /ESP32/EN -> GND
- U4 pad 4: /ESP32/~{JTAG_EN} -> /ESP32/USB_D+
- U4 pad 5: /ESP32/~{SBC3_FLT} -> /ESP32/USB_D-
- U4 pad 6: /ESP32/~{SBC2_FLT} -> +3V3
- U4 pad 7: /ESP32/~{SBC1_FLT} -> +3V3
- U4 pad 8: /ESP32/~{SBC1_EN} -> Net-(U4-VBUS)
- U4 pad 9: /ESP32/~{SBC2_EN} -> Net-(U4-~{RST})
- U8 pad 4: /ESP32/MTDO -> /ESP32/~{SBC3_EN}
- U9 pad 1: /Outputs/IN3- -> /Outputs/IN1-
- U9 pad 11: /Outputs/IN1- -> /Outputs/IN3-
- U9 pad 12: /Outputs/IN1+ -> /Outputs/IN3+
- U9 pad 2: /Outputs/IN3+ -> /Outputs/IN1+
- U9 pad 9: unconnected-(U9-CRITICAL-Pad9) -> /ESP32/CRITICAL
Routing:
- net /ESP32/SBC1_BTN: track 0.00 -> 100.2 mm, vias 0 -> 1
- net /ESP32/MTCK: track 85.2 -> 9.30 mm, vias 1 -> 0
- net +3V3: track 294.7 -> 358.3 mm, vias 12 -> 6
- net /ESP32/CRITICAL: track 0.00 -> 62.5 mm
- net +5V: track 145.6 -> 84.2 mm, vias 0 -> 2
- net /ESP32/~{SBC1_FLT}: track 88.7 -> 145.6 mm, vias 3 -> 1
- net /ESP32/~{SBC3_EN}: track 0.00 -> 54.2 mm, vias 0 -> 3
- net /ESP32/SBC2_BTN: track 0.00 -> 53.9 mm, vias 0 -> 1
- net /ESP32/~{SBC3_FLT}: track 28.7 -> 81.5 mm
- net /ESP32/MTDI: track 58.9 -> 8.79 mm, vias 3 -> 0
- net /ESP32/SBC3_BTN: track 0.00 -> 47.8 mm, vias 0 -> 1
- net /ESP32/MTMS: track 68.0 -> 22.0 mm, vias 2 -> 1
- net /Ethernet/LED2: track 35.9 -> 0.00 mm
- net /ESP32/RMII_RXD1: track 35.7 -> 0.00 mm, vias 2 -> 0
- net /ESP32/MTDO: track 45.7 -> 10.7 mm, vias 1 -> 0
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- added copper zone on F.Cu, net +5V
- removed copper zone on F.Cu, net +3V3_RegIn
- removed copper zone on F.Cu, net Net-(J5-VBUS)
- removed copper zone on F.Cu, net Net-(J6-VBUS)
- removed copper zone on F.Cu, net Net-(J7-VBUS)
Other:
- board text added: "+12V"
- board text added: "+3,3V"
- board text added: "+5V"
- board text added: "Button"
- board text added: "Reset"
- board text added: "SBC-PDU 1.0 rev 3 © 2023 Roman Ondráček sbc-pdu.romanondracek.cz MAC:"
- board text removed: "SBC-PDU 1.0 rev. 2 © 2023 Roman Ondráček"

Commit message: Fix third revision
Signed-off-by: Roman Ondráček <ondracek.roman@centrum.cz>
Parts:
- R21, R27, R34: value 100R -> 430R
- R22, R29, R35: value 100R -> 1k
Connections:
- U4 pad 25: /ESP32/DEBUG_RX -> /ESP32/DEBUG_TX
- U4 pad 26: /ESP32/DEBUG_TX -> /ESP32/DEBUG_RX
Routing:
- net GND: track 130.4 -> 108.3 mm
- net /ESP32/SBC2_BTN: track 53.9 -> 45.6 mm
- net /ESP32/SBC3_BTN: track 47.8 -> 39.9 mm
- net /ESP32/SBC1_BTN: track 100.2 -> 92.2 mm
- net /ESP32/~{SBC3_EN}: track 54.2 -> 49.0 mm
- net /ESP32/~{SBC2_FLT}: track 96.5 -> 92.3 mm, vias 1 -> 3
- net /ESP32/~{SBC1_FLT}: track 145.6 -> 141.5 mm, vias 1 -> 3
- net /ESP32/DEBUG_RX: track 66.2 -> 68.7 mm, vias 1 -> 3
- net Net-(D13-A): track 3.86 -> 5.83 mm
- net /Outputs/SBC1_POWER: track 18.7 -> 18.2 mm
