File: power.kicad_sch (KiCad schematic)
At the start: 27 parts, among them J1 Wuerth_694108301002, Q1 FDD4243, U1 LD1117S33TR_SOT223, U2 MAX17634BATP+

Commit message: Second revision
Signed-off-by: Roman Ondráček <ondracek.roman@centrum.cz>
Parts:
- added D2, D3: Green_LED, LED_SMD:LED_0603_1608Metric_Pad1.05x0.95mm_HandSolder, symbol Device:LED
- added D4: Amber_LED, LED_SMD:LED_0603_1608Metric_Pad1.05x0.95mm_HandSolder, symbol Device:LED
- added R3: 430R, Resistor_SMD:R_0603_1608Metric_Pad0.98x0.95mm_HandSolder, symbol Device:R
- added R4, R5: 100R, Resistor_SMD:R_0603_1608Metric_Pad0.98x0.95mm_HandSolder, symbol Device:R
- C1: renamed from C12; Mouser (none) -> https://cz.mouser.com/ProductDetail/187-CL21B104KCFSFNE
- C10: Mouser (none) -> https://cz.mouser.com/ProductDetail/81-GRM1555C1H562GE1D
- C11: Mouser (none) -> https://cz.mouser.com/ProductDetail/81-GRM188R71A225KE5J
- C12: renamed from C1; Mouser (none) -> https://cz.mouser.com/ProductDetail/187-CL10A105KA8NNNC
- C13: renamed from C2; Mouser (none) -> https://cz.mouser.com/ProductDetail/187-CL21B104KCFSFNE
- C14: renamed from C3; Mouser (none) -> https://cz.mouser.com/ProductDetail/81-GRM188R61A106ME9D
- C2: renamed from C5; Mouser (none) -> https://cz.mouser.com/ProductDetail/647-UCM1H470MCL1GS
- C3: renamed from C6; Mouser (none) -> https://cz.mouser.com/ProductDetail/81-GRM31CR71H475KA2K
- C4: renamed from C7; Mouser (none) -> https://cz.mouser.com/ProductDetail/81-GRM31CR71H475KA2K
- C5: renamed from C8; Mouser (none) -> https://cz.mouser.com/ProductDetail/810-C1005C0G2A151JBA
- C6: renamed from C9; Mouser (none) -> https://cz.mouser.com/ProductDetail/810-C1005C0G2A151JBA
- C8: renamed from C13; Mouser (none) -> https://cz.mouser.com/ProductDetail/81-GRM32ER71A476ME5L
- C9: renamed from C14; Mouser (none) -> https://cz.mouser.com/ProductDetail/81-GRM32ER71A476ME5L
- D1: Mouser (none) -> https://cz.mouser.com/ProductDetail/78-SMAJ12CAHE3_A-H
- F1: Mouser (none) -> https://cz.mouser.com/ProductDetail/530-C1T5
- J1: value Wuerth_694108301002 -> DC_Jack; footprint Connector_BarrelJack:BarrelJack_Wuerth_6941xx301002 -> Connector_BarrelJack:BarrelJack_Horizontal; Mouser (none) -> https://cz.mouser.com/ProductDetail/161-0725-E
- L1: value 8.2uH -> 8.2u; footprint Inductor_SMD:L_Bourns_SRP1245A -> Inductor_SMD:L_Coilcraft_XAL6060-XXX; Mouser (none) -> https://cz.mouser.com/ProductDetail/Coilcraft/XAL6060-822MEC
- Q1: Mouser (none) -> https://cz.mouser.com/ProductDetail/512-FDD4243
- R1: Mouser (none) -> https://cz.mouser.com/ProductDetail/667-ERJ-2RKF5102X
- R2: Mouser (none) -> https://cz.mouser.com/ProductDetail/652-CR0402FX-1002GLF
- U1: renamed from U2; footprint Package_DFN_QFN_custom:TQFN-20-1EP_4x4mm_P0.5mm_EP2.9x2.9mm -> Package_DFN_QFN:TQFN-20-1EP_4x4mm_P0.5mm_EP2.9x2.9mm; Mouser (none) -> https://cz.mouser.com/ProductDetail/700-MAX17634BATP%2b
- U2: renamed from U1; value LD1117S33TR_SOT223 -> TLV1117LV33DCYR; Mouser (none) -> https://cz.mouser.com/ProductDetail/595-TLV1117LV33DCYR
- renumbered C4 to C7
Connections:
- net +12V: now also R3.1
- net +3V3: now also R5.1
- net +5V: now also R4.1
- net GND: now also D2.1 (K), D3.1 (K), D4.1 (K)
- net Vin: now reaches D1.2 (A2), F1.2, Q1.2 (D)
- new net: D3.2 (A), R4.2
- new net: D2.2 (A), R3.2
- new net: D4.2 (A), R5.2
Other:
- title: (none) -> PDU with Consumption Metering Function for SBCs
- moved on the sheet: C1, C10, C11, C2, C3, C4, C5, C6, C8, C9, L1, R1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

Commit message: Third revision
Signed-off-by: Roman Ondráček <ondracek.roman@centrum.cz>
Parts:
- L1: footprint Inductor_SMD:L_Coilcraft_XAL6060-XXX -> Inductor_SMD:L_Bourns_SRP1245A
- R4, R5: value 100R -> 430R
Other:
- note added: "Test LEDs"
- moved on the sheet: D2, D3, D4, R3, R4, R5, TP1, TP2, TP3, TP4

Commit message: Fix third revision
Signed-off-by: Roman Ondráček <ondracek.roman@centrum.cz>
Parts:
- C1, C13: Mouser https://cz.mouser.com/ProductDetail/187-CL21B104KCFSFNE -> https://cz.mouser.com/ProductDetail/81-GRM155R62A104KE4J
- C7: Mouser (none) -> https://cz.mouser.com/ProductDetail/647-UVR1C471MPD
- J1: Mouser https://cz.mouser.com/ProductDetail/161-0725-E -> (none); TME (none) -> https://www.tme.eu/cz/details/fc68148/konektory-dc/cliff/dc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
Other:
- moved on the sheet: C1, C10, C11, C2, C3, C4, C5, C6, C8, C9, L1, R1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
